Commit message: changed orientation of alpha arm; PID tuned

File: urdf/alpha_seabotix.urdf (robot description, URDF)
Before this commit: robot uvms_alpha_seabotix, 28 links, 27 joints
Joints:
- joint arm_to_vehicle: origin xyz=.45 0 0 rpy=3.1415 0 0 -> xyz=.325 0 -.09 rpy=3.1415 0 0
- joint r5m_joint4: origin xyz=0.020 0 0.046 rpy=1.57075 -0.27079 0 -> xyz=0.020 0 0.046 rpy=1.57075 1.3 0
- joint r5m_joint5: origin xyz=0 0 0 rpy=0 0 3.141592 -> xyz=0 0 0 rpy=0 0 0

Commit message: Check that cob and com frames are right

File: urdf/alpha_seabotix.urdf (robot description, URDF)
Before this commit: robot uvms_alpha_seabotix, 28 links, 27 joints
Links:
- link r5m_jaw2: mass 0.5 -> 0.05
