Commit message: alpha attached to URDF (not final config)

File: urdf/blue_rov.urdf (robot description, URDF)
Before this commit: robot bluerov, 3 links, 2 joints
Links:
- added link r5m_base_link, mass 0.53; collision cylinder length=0.150 radius=0.020; visual mesh filename=C:\Users\hkola\Stuff\_ONR\RNNs for pitch prediction\PitchPr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
- added link r5m_forearm_link, mass 0.147; collision cylinder length=0.040 radius=0.020; visual mesh filename=C:\Users\hkola\Stuff\_ONR\RNNs for pitch prediction\PitchPr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
- added link r5m_jaw
- added link r5m_jaw1, mass 0.05; collision box size=0.03 0.09 0.01; visual mesh filename=C:\Users\hkola\Stuff\_ONR\RNNs for pitch prediction\PitchPr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
- added link r5m_jaw2, mass 0.05; collision box size=0.03 0.09 0.01; visual mesh filename=C:\Users\hkola\Stuff\_ONR\RNNs for pitch prediction\PitchPr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
- added link r5m_shoulder_link, mass 0.226; collision cylinder length=0.066 radius=0.020; visual mesh filename=C:\Users\hkola\Stuff\_ONR\RNNs for pitch prediction\PitchPr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
- added link r5m_upper_arm_link, mass 0.630; collision cylinder length=0.040 radius=0.020; collision cylinder length=0.145 radius=0.020
- added link r5m_wrist_link, mass 0.559; collision cylinder length=0.140 radius=0.020; visual mesh filename=C:\Users\hkola\Stuff\_ONR\RNNs for pitch prediction\PitchPr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
Joints:
- added joint arm_to_vehicle: type fixed, parent vehicle_frame, child r5m_base_link, origin xyz=.15 0 -.15 rpy=3.1415 0 0
- added joint r5m_joint1_1: type fixed, parent r5m_wrist_link, child r5m_jaw2, origin xyz=-0.015 0 -0.140 rpy=1.57075 0 0, axis 0 0 -1, limit lower=0.0 upper=0.5 effort=5.0 velocity=0.5
- added joint r5m_joint1_2: type fixed, parent r5m_wrist_link, child r5m_jaw1, origin xyz=0.015 0 -0.140 rpy=1.57075 0 0, axis 0 0 1, limit lower=0.0 upper=0.5 effort=5.0 velocity=0.5
- added joint r5m_joint2: type revolute, parent r5m_forearm_link, child r5m_wrist_link, origin xyz=0.020 0 0 rpy=-1.57075 -0.5 0, axis 0 0 1, limit lower=0.0 upper=6.0 effort=5.0 velocity=1.0
- added joint r5m_joint3: type revolute, parent r5m_upper_arm_link, child r5m_forearm_link, origin xyz=0.15 0 0 rpy=3.1415 0 1.3, axis 0 0 1, limit lower=0.0 upper=3.5 effort=9.0 velocity=0.5
- added joint r5m_joint4: type revolute, parent r5m_shoulder_link, child r5m_upper_arm_link, origin xyz=0.020 0 0.046 rpy=1.57075 1.3 0, axis 0 0 1, limit lower=0.0 upper=3.5 effort=9.0 velocity=0.5
- added joint r5m_joint5: type revolute, parent r5m_base_link, child r5m_shoulder_link, origin xyz=0 0 0 rpy=0 0 0, axis 0 0 1, limit lower=0.0 upper=6.2 effort=9.0 velocity=0.5
- added joint r5m_joint_jaw: type fixed, parent r5m_wrist_link, child r5m_jaw, origin xyz=0 0 -0.190 rpy=0 0 1.5707

Commit message: added extra link to URDF for extra frame, partial functionality

File: urdf/blue_rov.urdf (robot description, URDF)
Before this commit: robot bluerov, 11 links, 10 joints
Joints:
- joint r5m_joint_jaw: axis (none) -> 0 0 1; origin xyz=0 0 -0.190 rpy=0 0 1.5707 -> xyz=0 0 -0.190 rpy=0 0 0; type fixed -> prismatic

Commit message: added jaw link to sim. Not yet actuated.

File: urdf/blue_rov.urdf (robot description, URDF)
Before this commit: robot bluerov, 11 links, 10 joints
Links:
- link r5m_jaw: mass None -> 0.01

Commit message: updated packages; fixed twist of wrist

File: urdf/blue_rov.urdf (robot description, URDF)
Before this commit: robot bluerov, 11 links, 10 joints
Joints:
- joint r5m_joint2: origin xyz=0.020 0 0 rpy=-1.57075 -0.5 0 -> xyz=0.020 0 0 rpy=-1.57075 0.0 0

Commit message: change jaw joint to prismatic

File: urdf/blue_rov.urdf (robot description, URDF)
Before this commit: robot bluerov, 11 links, 10 joints
Joints:
- joint r5m_joint1_1: origin xyz=-0.015 0 -0.140 rpy=1.57075 0 0 -> xyz=-0.015 0 .05 rpy=1.57075 0 0; parent r5m_wrist_link -> r5m_jaw
- joint r5m_joint1_2: origin xyz=0.015 0 -0.140 rpy=1.57075 0 0 -> xyz=0.015 0 .05 rpy=1.57075 0 0; parent r5m_wrist_link -> r5m_jaw
- joint r5m_joint_jaw: type prismatic -> revolute

Commit message: Added back Random, Rotations packages

File: urdf/blue_rov.urdf (robot description, URDF)
Before this commit: robot bluerov, 11 links, 10 joints
Joints:
- joint r5m_joint_jaw: type prismatic -> revolute

Commit message: separate TrajGen funcs, merge urdf changes for jaw joint

File: urdf/blue_rov.urdf (robot description, URDF)
Before this commit: robot bluerov, 11 links, 10 joints
Joints:
- joint r5m_joint1_1: origin xyz=-0.015 0 -0.140 rpy=1.57075 0 0 -> xyz=-0.015 0 .05 rpy=1.57075 0 0; parent r5m_wrist_link -> r5m_jaw
- joint r5m_joint1_2: origin xyz=0.015 0 -0.140 rpy=1.57075 0 0 -> xyz=0.015 0 .05 rpy=1.57075 0 0; parent r5m_wrist_link -> r5m_jaw

Commit message: back to joint trajectories

File: urdf/blue_rov.urdf (robot description, URDF)
Before this commit: robot bluerov, 11 links, 10 joints
Joints:
- joint r5m_joint_jaw: type revolute -> fixed

Commit message: relative OBJ paths; ignoring jaw joint for pitch pred

File: urdf/blue_rov.urdf (robot description, URDF)
Before this commit: robot bluerov, 11 links, 10 joints
Links:
- link r5m_base_link: geometry collision cylinder length=0.150 radius=0.020; visual mesh filename=meshes\Base3.obj
- link r5m_forearm_link: geometry collision cylinder length=0.040 radius=0.020; visual mesh filename=meshes\ElbowJoint3.obj
- link r5m_jaw1: geometry collision box size=0.03 0.09 0.01; visual mesh filename=meshes\Jaw1_v2.obj
- link r5m_jaw2: geometry collision box size=0.03 0.09 0.01; visual mesh filename=meshes\Jaw2_v2.obj
- link r5m_shoulder_link: geometry collision cylinder length=0.066 radius=0.020; visual mesh filename=meshes\ShoulderJoint3.obj
- link r5m_upper_arm_link: geometry collision cylinder length=0.040 radius=0.020; collision cylinder length=0.145 radius=0.020
- link r5m_wrist_link: geometry collision cylinder length=0.140 radius=0.020; visual mesh filename=meshes\Wrist3.obj
- link vehicle_ballast: geometry visual mesh filename=meshes\bluerov_blue.obj
- link vehicle_cans: geometry visual mesh filename=meshes\bluerov_white.obj
- link vehicle_frame: geometry visual mesh filename=meshes\bluerov_black.obj
