Commit message: upload traj files that were used in hinsdale testing

File: urdf/blue_rov_hardware.urdf (robot description, URDF)
Before this commit: robot bluerov, 11 links, 10 joints
Links:
- link r5m_base_link: geometry collision cylinder length=0.150 radius=0.020; visual mesh filename=meshes/Base3.obj
- link r5m_forearm_link: geometry collision cylinder length=0.040 radius=0.020; visual mesh filename=meshes/ElbowJoint3.obj
- link r5m_jaw1: geometry collision box size=0.03 0.09 0.01; visual mesh filename=meshes/Jaw1_v2.obj
- link r5m_jaw2: geometry collision box size=0.03 0.09 0.01; visual mesh filename=meshes/Jaw2_v2.obj
- link r5m_shoulder_link: geometry collision cylinder length=0.066 radius=0.020; visual mesh filename=meshes/ShoulderJoint3.obj
- link r5m_upper_arm_link: geometry collision cylinder length=0.040 radius=0.020; collision cylinder length=0.145 radius=0.020
- link r5m_wrist_link: geometry collision cylinder length=0.140 radius=0.020; visual mesh filename=meshes/Wrist3.obj
- link vehicle_ballast: geometry visual mesh filename=meshes/bluerov_blue.obj
- link vehicle_cans: geometry visual mesh filename=meshes/bluerov_white.obj
- link vehicle_frame: geometry visual mesh filename=meshes/bluerov_black.obj

Commit message: tweaks to make no-arm behavior similar in sim and hinsdale

File: urdf/blue_rov_hardware.urdf (robot description, URDF)
Before this commit: robot bluerov, 11 links, 10 joints
Links:
- link vehicle_frame: mass 20.9 -> 25.14
Joints:
- joint arm_to_vehicle: origin xyz=.255 -.10965 0.005 rpy=0 0 0 -> xyz=.25 -.10965 0.005 rpy=0 0 0
